Commit message: Addopting Jetbot Box Model

File: urdf/includes/parts/antenna.xacro (robot description, xacro)
@@ -10,7 +10,4 @@
   <xacro:property name="antenna_top_mass" value="0.06" /-->
   <!-- Antenna constants -->
-  <!-- Inertia Macros -->
-  <xacro:include filename="$(find jetbot_ccai)/urdf/includes/gazebo/inertias.xacro" />
-  <!-- Inertia Macros -->
   <!-- Left and Right Antenna Macro -->
   <xacro:macro name="antenna" params="prefix reflect">
@@ -29,5 +26,4 @@
       </geometry>
     </collision>
-    <xacro:cylinder_inertia mass="${antenna_body_mass}" r="${antenna_r}" h="${antenna_len}" />
   </link>
   <joint name="base_${prefix}_antenna_joint" type="fixed">
@@ -48,5 +44,4 @@
       </geometry>
     </collision>
-    <xacro:sphere_inertia mass="${antenna_top_mass}" r="${antenna_r}" />
   </link>
   <joint name="${prefix}_antenna_top_joint" type="fixed">

File: urdf/includes/parts/boards.xacro (robot description, xacro)
@@ -8,28 +8,24 @@
   <!--xacro:property name="box_mass" value="0.6" /-->
   <!-- Motor driver and PCB constants -->
-  <!-- Inertias Macros -->
-  <xacro:include filename="$(find jetbot_ccai)/urdf/includes/gazebo/inertias.xacro" />
-  <!-- Inertias Macros -->
   <!-- PCB, MOTOR DRIVER AND JETSON NANO -->
   <xacro:macro name="pcb">
-  <link name="pcb_boards">
-    <visual>
-      <geometry>
-        <box size="${box_len} ${box_width} ${box_height}"/>
-      </geometry>
-      <material name="green"/>
-    </visual>
-    <collision>
-      <geometry>
-        <box size="${box_len} ${box_width} ${box_height}"/>
-      </geometry>
-    </collision>
-    <xacro:cuboid_inertia mass="${box_mass}" x="${box_len}" y="${box_width}" z="${box_height}" />
-  </link>
-  <joint name="base_nano_joint" type="fixed">
-    <parent link="base_link"/>
-    <child link="pcb_boards"/>
-    <origin xyz="0 0 ${box_height}"/>
-  </joint>
+    <link name="pcb_boards">
+      <visual>
+        <geometry>
+          <box size="${box_len} ${box_width} ${box_height}"/>
+        </geometry>
+        <material name="green"/>
+      </visual>
+      <collision>
+        <geometry>
+          <box size="${box_len} ${box_width} ${box_height}"/>
+        </geometry>
+      </collision>
+    </link>
+    <joint name="base_nano_joint" type="fixed">
+      <parent link="base_link"/>
+      <child link="pcb_boards"/>
+      <origin xyz="0 0 ${box_height}"/>
+    </joint>
   </xacro:macro>
   <!-- PCB, MOTOR DRIVER AND JETSON NANO -->

File: urdf/includes/parts/camera.xacro (robot description, xacro)
@@ -1,7 +1,4 @@
 <?xml version="1.0"?>
 <robot xmlns:xacro="http://www.ros.org/wiki/xacro">
-<!-- Inertias Macros -->
-<xacro:include filename="$(find jetbot_ccai)/urdf/includes/gazebo/inertias.xacro" />
-<!-- Inertias Macros -->
 <xacro:property name="camera_mount_base_mass" value="0.01" />
 <xacro:property name="camera_mount_over_mass" value="0.005" />
@@ -29,5 +26,4 @@
       </geometry>
     </collision>
-    <xacro:cuboid_inertia mass="${camera_mount_base_mass}" x="0.01" y="0.04" z="0.002" />
   </link>
   <joint name="camera_mount_base_joint" type="fixed">
@@ -50,5 +46,4 @@
       </geometry>
     </collision>
-    <xacro:cuboid_inertia mass="${camera_mount_over_mass}" x="0.03" y="0.04" z="0.002"/>
   </link>
   <joint name="camera_mount_over_joint" type="fixed">
@@ -71,5 +66,4 @@
       </geometry>
     </collision>
-    <xacro:cuboid_inertia mass="${camera_mount_angled_mass}" x="0.025" y="0.025" z="0.002" />
   </link>
   <joint name="camera_mount_angled_joint" type="fixed">
@@ -92,5 +86,4 @@
       </geometry>
     </collision>
-    <xacro:cuboid_inertia mass="${camera_screen_base_mass}" x="0.025" y="0.025" z="0.004" />
   </link>
   <joint name="camera_mount_screen_joint" type="fixed">
@@ -113,5 +106,4 @@
       </geometry>
     </collision>
-    <xacro:cuboid_inertia mass="${camera_pcb_base_mass}" x="0.013" y="0.013" z="0.004" />
   </link>
   <joint name="camera_pcb_base_joint" type="fixed">
@@ -134,5 +126,4 @@
       </geometry>
     </collision>
-    <xacro:cylinder_inertia mass="${camera_lens_body_mass}" r="0.006" h="0.01" />
   </link>
   <joint name="camera_lens_body_joint" type="fixed">
@@ -155,5 +146,4 @@
       </geometry>
     </collision>
-    <xacro:cylinder_inertia mass="${camera_lens_body_out_mass}" r="0.0075" h="0.003"/>
   </link>
  <joint name="camera_lens_body_out_joint" type="fixed">
@@ -176,5 +166,4 @@
       </geometry>
     </collision>
-    <xacro:sphere_inertia mass="${camera_lens_mass}" r="0.005" />
   </link>
  <joint name="camera_lens_joint" type="fixed">

File: urdf/includes/parts/chassis.xacro (robot description, xacro)
@@ -10,27 +10,26 @@
   <!-- Chassis constants -->
   <!-- CHASSIS (body) -->
-  <xacro:macro name="chassis" >
-  <link name="base_footprint" />
-  <link name="base_link">
-    <visual>
-      <origin xyz="0 0 ${base_z_offset}"/>
-      <geometry>
-        <box size="${base_len} ${base_width} ${base_height}"/>
-      </geometry>
-      <material name="blue"/>
-    </visual>
-    <collision>
-      <origin xyz="0 0 ${base_z_offset}"/>
-      <geometry>
-        <box size="${base_len} ${base_width} ${base_height}"/>
-      </geometry>
-    </collision>
-    <xacro:cuboid_inertia mass="${base_mass}" x="${base_len}" y="${base_width}" z="${base_height}" />
-  </link>
-  <!-- Joint to connect base_link with base_footprint -->
-  <joint name="base_footprint_joint" type="fixed">
-    <parent link="base_footprint"/>
-    <child link="base_link" />
-  </joint>
+  <xacro:macro name="chassis">
+    <!--link name="base_footprint" /-->
+    <link name="base_link">
+      <visual>
+        <origin xyz="0 0 ${base_z_offset}"/>
+        <geometry>
+          <box size="${base_len} ${base_width} ${base_height}"/>
+        </geometry>
+        <material name="blue"/>
+      </visual>
+      <collision>
+        <origin xyz="0 0 ${base_z_offset}"/>
+        <geometry>
+          <box size="${base_len} ${base_width} ${base_height}"/>
+        </geometry>
+      </collision>
+    </link>
+    <!-- Joint to connect base_link with base_footprint >
+    <joint name="base_footprint_joint" type="fixed">
+      <parent link="base_footprint"/>
+      <child link="base_link" />
+    </joint-->
   </xacro:macro>
   <!-- CHASSIS (body) -->

File: urdf/includes/parts/sensors/laser/laser.urdf.xacro (robot description, xacro)
@@ -23,11 +23,4 @@
         </geometry>
       </collision>
-      <inertial>
-        <mass value="0.114" />
-        <origin xyz="0 0 0" />
-        <inertia ixx="0.001" ixy="0.0" ixz="0.0"
-                 iyy="0.001" iyz="0.0"
-                 izz="0.001" />
-      </inertial>
     </link>
     <!-- RPLidar Plugin -->

File: urdf/includes/parts/sensors/rgbcam/camera.xacro (robot description, xacro)
@@ -1,7 +1,4 @@
 <?xml version="1.0"?>
 <robot xmlns:xacro="http://www.ros.org/wiki/xacro">
-<!-- Inertias Macros -->
-<xacro:include filename="$(find jetbot_ccai)/urdf/includes/gazebo/inertias.xacro" />
-<!-- Inertias Macros -->
 <!-- CAMERA -->
  <xacro:macro name="camera" >
@@ -18,5 +15,4 @@
       </geometry>
     </collision>
-    <xacro:cuboid_inertia mass="0.009" x="0.01" y="0.04" z="0.002" />
   </link>
   <joint name="camera_mount_base_joint" type="fixed">
@@ -39,5 +35,4 @@
       </geometry>
     </collision>
-    <xacro:cuboid_inertia mass="0.009" x="0.03" y="0.04" z="0.002"/>
   </link>
   <joint name="camera_mount_over_joint" type="fixed">
@@ -60,5 +55,4 @@
       </geometry>
     </collision>
-    <xacro:cuboid_inertia mass="0.009" x="0.025" y="0.025" z="0.002" />
   </link>
   <joint name="camera_mount_angled_joint" type="fixed">
@@ -81,5 +75,4 @@
       </geometry>
     </collision>
-    <xacro:cuboid_inertia mass="0.009" x="0.025" y="0.025" z="0.004" />
   </link>
   <joint name="camera_mount_screen_joint" type="fixed">
@@ -102,5 +95,4 @@
       </geometry>
     </collision>
-    <xacro:cuboid_inertia mass="0.009" x="0.013" y="0.013" z="0.004" />
   </link>
   <joint name="camera_pcb_base_joint" type="fixed">
@@ -123,5 +115,4 @@
       </geometry>
     </collision>
-    <xacro:cylinder_inertia mass="0.022" r="0.006" h="0.01" />
   </link>
   <joint name="camera_lens_body_joint" type="fixed">
@@ -144,5 +135,4 @@
       </geometry>
     </collision>
-    <xacro:cylinder_inertia mass="0.009" r="0.0075" h="0.003"/>
   </link>
  <joint name="camera_lens_body_out_joint" type="fixed">
@@ -165,5 +155,4 @@
       </geometry>
     </collision>
-    <xacro:sphere_inertia mass="0.006" r="0.005" />
   </link>
  <joint name="camera_lens_joint" type="fixed">

File: urdf/includes/parts/wheels/caster.xacro (robot description, xacro)
@@ -12,7 +12,4 @@
   <xacro:property name="caster_ball_mass" value="0.02" />
   <!-- Caster Ball constants -->
-  <!-- Inertia Macro -->
-  <xacro:include filename="$(find jetbot_ccai)/urdf/includes/gazebo/inertias.xacro" />
-  <!-- Inertia Macro -->
   <!-- Caster Wheel Left and Right Mini Cylinder Macros -->
   <xacro:macro name="caster_minicyl" params="prefix suffix reflect">
@@ -29,5 +26,4 @@
       </geometry>
     </collision>
-    <xacro:cylinder_inertia mass="${caster_minicyl_mass}" r="${caster_cyl_r/3.75}" h="${caster_cyl_len}" />
   </link>
   <joint name="${prefix}_caster_${suffix}_cyl_joint" type="fixed">
@@ -52,5 +48,4 @@
       </geometry>
     </collision>
-    <xacro:cylinder_inertia mass="${caster_cyl_mass}" r="${caster_cyl_r}" h="${caster_cyl_len}" />
   </link>
   <joint name="base_${prefix}_caster_joint" type="fixed">
@@ -73,5 +68,4 @@
       </geometry>
     </collision>
-    <xacro:sphere_inertia mass="${caster_ball_mass}" r="${caster_ball}" />
   </link>
   <joint name="${prefix}_caster_joint" type="fixed">

File: urdf/includes/parts/wheels/wheel.xacro (robot description, xacro)
@@ -8,58 +8,56 @@
   <xacro:property name="wheelc_len" value="0.015" />
   <xacro:property name="wheelc_r" value = "0.026" />
-  <xacro:property name="wheel_shaft_mass" value = "0.000283495" /> <!--0.000283495 0.0028 -->
-  <xacro:property name="wheelc_mass" value = "0.283495" />  <!--0.283495 0.00283495 0.0272 -->
-  <xacro:property name="wheel_mass" value = "0.0181" />         <!--3.0 0.0181 -->
+  <xacro:property name="wheel_shaft_mass" value = "0.000283495" />
+  <!--0.000283495 0.0028 -->
+  <xacro:property name="wheelc_mass" value = "0.283495" />
+  <!--0.283495 0.00283495 0.0272 -->
+  <xacro:property name="wheel_mass" value = "0.0181" />
+  <!--3.0 0.0181 -->
   <!-- Wheel constants -->
-  <!-- Inertia Macro -->
-  <xacro:include filename="$(find jetbot_ccai)/urdf/includes/gazebo/inertias.xacro" />
-  <!-- Inertia Macro -->
   <!-- Wheel Macro-->
   <xacro:macro name="wheel_parts" params="prefix reflect">
-  <link name="${prefix}_wheel_shaft">
-    <visual>
-      <origin xyz="0 0 0" rpy="${pi/2} 0 0"/>
-      <geometry>
-        <cylinder radius="${shaft_r}" length="${shaft_len}" />
-      </geometry>
-      <material name="white"/>
-    </visual>
-    <collision>
-      <origin xyz="0 0 0" rpy="${pi/2} 0 0"/>
-      <geometry>
-        <cylinder radius="${shaft_r}" length="${shaft_len}" />
-      </geometry>
-    </collision>
-    <xacro:cylinder_inertia mass="${wheel_shaft_mass}" r="${shaft_r}" h="${shaft_len}"/>
-  </link>
-  <joint name="base_${prefix}_wheel_shaft_joint" type="fixed">
-    <axis rpy="0 0 0" xyz="0 0 0" />
-    <parent link="base_link"/>
-    <child link="${prefix}_wheel_shaft"/>
-    <origin rpy="0 0 0" xyz="${shaft_xoffset} ${shaft_yoffset*reflect} 0.013" />
-  </joint>
-  <link name="${prefix}_wheelc">
-    <visual>
-      <origin rpy="${pi/2} 0 0"/>
-      <geometry>
-        <cylinder length="${wheelc_len}" radius="${wheelc_r}"/>
-      </geometry>
-      <material name="white"/>
-    </visual>
-    <collision>
-      <origin rpy="${pi/2} 0 0"/>
-      <geometry>
-        <cylinder length="${wheelc_len}" radius="${wheelc_r}"/>
-      </geometry>
-    </collision>
-    <xacro:inertia mass="0.6" />
-    <!--xacro:cylinder_inertia mass="${wheelc_mass}" r="${wheelc_r}" h="${wheelc_len}" /-->
-  </link>
-  <joint name="${prefix}_shaft_wheelc_joint" type="fixed">
-    <origin xyz="0 ${reflect*(wheelc_r-0.002)/2} 0"/>
-    <parent link="${prefix}_wheel_shaft"/>
-    <child link="${prefix}_wheelc"/>
-  </joint>
-  <link name="${prefix}_wheel">
+    <link name="${prefix}_wheel_shaft">
+      <visual>
+        <origin xyz="0 0 0" rpy="${pi/2} 0 0"/>
+        <geometry>
+          <cylinder radius="${shaft_r}" length="${shaft_len}" />
+        </geometry>
+        <material name="white"/>
+      </visual>
+      <collision>
+        <origin xyz="0 0 0" rpy="${pi/2} 0 0"/>
+        <geometry>
+          <cylinder radius="${shaft_r}" length="${shaft_len}" />
+        </geometry>
+      </collision>
+    </link>
+    <joint name="base_${prefix}_wheel_shaft_joint" type="fixed">
+      <axis rpy="0 0 0" xyz="0 0 0" />
+      <parent link="base_link"/>
+      <child link="${prefix}_wheel_shaft"/>
+      <origin rpy="0 0 0" xyz="${shaft_xoffset} ${shaft_yoffset*reflect} 0.013" />
+    </joint>
+    <link name="${prefix}_wheelc">
+      <visual>
+        <origin rpy="${pi/2} 0 0"/>
+        <geometry>
+          <cylinder length="${wheelc_len}" radius="${wheelc_r}"/>
+        </geometry>
+        <material name="white"/>
+      </visual>
+      <collision>
+        <origin rpy="${pi/2} 0 0"/>
+        <geometry>
+          <cylinder length="${wheelc_len}" radius="${wheelc_r}"/>
+        </geometry>
+      </collision>
+      <!--xacro:cylinder_inertia mass="${wheelc_mass}" r="${wheelc_r}" h="${wheelc_len}" /-->
+    </link>
+    <joint name="${prefix}_shaft_wheelc_joint" type="fixed">
+      <origin xyz="0 ${reflect*(wheelc_r-0.002)/2} 0"/>
+      <parent link="${prefix}_wheel_shaft"/>
+      <child link="${prefix}_wheelc"/>
+    </joint>
+    <!--link name="${prefix}_wheel">
     <visual>
     <origin rpy="${pi/2} 0 0" xyz="0 0 0" />
@@ -75,6 +73,4 @@
       </geometry>
     </collision>
-    <xacro:inertia mass="0.6"/>
-    <!--xacro:open_cylinder_inertia mass="${wheel_mass}" r1="${wheelc_r}" r2="${wheelc_r + 0.0065}" h="${wheelc_len}" /-->
   </link>
   <joint name="${prefix}_wheel_joint" type="continuous">
@@ -84,5 +80,5 @@
     <origin xyz ="0 ${-0.0001*reflect} 0"/>
   </joint>
-  <xacro:tx prefix="${prefix}" suffix="wheel" />
+    <xacro:tx prefix="${prefix}" suffix="wheel" /-->
   </xacro:macro>
   <!-- Wheel Macro-->

File: urdf/jetbot.urdf.xacro (robot description, xacro)
@@ -2,15 +2,15 @@
 <robot xmlns:xacro="http://www.ros.org/wiki/xacro" name="mobile_robot" >
   <!-- Xacro arguments for depth camera use -->
-  <xacro:arg name="realsense_enable" default="true" />
-  <xacro:arg name="pointcloud_enable" default="true" />
+  <xacro:arg name="realsense_enable" default="false" />
+  <xacro:arg name="pointcloud_enable" default="false" />
   <!-- Xacro arguments for depth lidar use -->
   <xacro:arg name="lidar_enable" default="true" />
   <xacro:arg name="visualize_laser" default="true" />
   <!-- Xacro arguments for imu -->
-  <xacro:arg name="imu_enable" default="true" />
+  <xacro:arg name="imu_enable" default="false" />
   <!-- Xacro arguments for gps -->
-  <xacro:arg name="gps_enable" default="true" />
+  <xacro:arg name="gps_enable" default="false" />
   <!-- Xacro arguments for ultrasonic -->
-  <xacro:arg name="ultrasonic_enable" default="true" />
+  <xacro:arg name="ultrasonic_enable" default="false" />
   <!-- All Neccesary Header Files, Macros and Constants -->
   <xacro:include filename="$(find jetbot_ccai)/urdf/includes.xacro" />
@@ -27,7 +27,7 @@
   <xacro:caster_wheel_parts prefix="back" reflect="-1" />
   <!-- LEFT ANTENNA -->
-  <xacro:antenna prefix="lt" reflect="1" />
+  <!--xacro:antenna prefix="lt" reflect="1" /-->
   <!-- RIGHT ANTENNA -->
-  <xacro:antenna prefix="rt" reflect="-1" />
+  <!--xacro:antenna prefix="rt" reflect="-1" /-->
   <!-- SENSORS -->
   <!-- MONOCULAR CAMERA -->
@@ -48,42 +48,3 @@
     </xacro:sensor_rplidar >
   </xacro:if>
-  <!-- IMU -->
-  <xacro:if value="$(arg imu_enable)" >
-    <xacro:sensor_imu name="imu" topic_ns="imu" parent="pcb_boards" >
-      <origin xyz="0 0 0.0275" rpy="0 0 0" />
-    </xacro:sensor_imu>
-  </xacro:if>
-  <!-- GPS -->
-  <xacro:if value="$(arg gps_enable)" >
-    <xacro:sensor_gps name="mtk3339" topic_ns="mtk_gps" parent="imu_link" >
-      <origin xyz="-0.044 0 0" rpy="0 0 0" />
-    </xacro:sensor_gps>
-  </xacro:if>
-  <!-- Ultrasonic Sensors -->
-  <xacro:if value="$(arg ultrasonic_enable)" >
-    <xacro:sensor_sonar name="sonar_1" topic_ns="sonar_back_rt" prefix="back_rt" parent="base_link" >
-      <origin xyz="-${base_len/3.5} -${base_width/2} ${base_height/2}" rpy="0 0 -${pi/2}" />
-    </xacro:sensor_sonar>
-    <xacro:sensor_sonar name="sonar_2" topic_ns="sonar_front_rt45" prefix="front_rt45" parent="base_link" >
-      <origin xyz="${base_len/2} -${base_width/2} ${base_height+(base_z_offset)/2}" rpy="0 0 -${pi/4}" />
-    </xacro:sensor_sonar>
-    <xacro:sensor_sonar name="sonar_3" topic_ns="sonar_front" prefix="front" parent="camera_mount_over" >
-      <origin xyz="0 0 0" rpy="0 0 0" />
-    </xacro:sensor_sonar>
-    <xacro:sensor_sonar name="sonar_4" topic_ns="sonar_front_lt45" prefix="front_lt45" parent="base_link" >
-      <origin xyz="${base_len/2} ${base_width/2} ${base_height+(base_z_offset)/2}" rpy="0 0 ${pi/4}" />
-    </xacro:sensor_sonar>
-    <xacro:sensor_sonar name="sonar_5" topic_ns="sonar_back_lt" prefix="back_lt" parent="base_link" >
-      <origin xyz="-${base_len/3.5} ${base_width/2} ${base_height/2}" rpy="0 0 ${pi/2}" />
-    </xacro:sensor_sonar>
-    <xacro:sensor_sonar name="sonar_6" topic_ns="sonar_back_lt45" prefix="back_lt45" parent="base_link" >
-      <origin xyz="-${base_len/2} ${base_width/2} ${base_height+(base_z_offset)/2}" rpy="0 0 ${pi/2 + pi/4}" />
-    </xacro:sensor_sonar>
-    <xacro:sensor_sonar name="sonar_7" topic_ns="sonar_back" prefix="back" parent="base_link" >
-      <origin xyz="-${base_len/2} 0 ${base_height/2}" rpy="0 0 ${pi}" />
-    </xacro:sensor_sonar>
-    <xacro:sensor_sonar name="sonar_8" topic_ns="sonar_back_rt45" prefix="back_rt45" parent="base_link" >
-      <origin xyz="-${base_len/2} -${base_width/2} ${base_height+(base_z_offset)/2}" rpy="0 0 -${pi/2 + pi/4}" />
-    </xacro:sensor_sonar>
-  </xacro:if>
 </robot>

File: urdf/mobile_robot.urdf.xacro (robot description, xacro)
@@ -1,42 +1,30 @@
 <?xml version="1.0"?>
-<robot name="mobile_robot" xmlns:xacro="http://ros.org/wiki/xacro">
-    <material name="blue">
-	    <color rgba="0 0 0.8 1"/>
-    </material>
-    <material name="white">
-	    <color rgba="1 1 1 1"/>
-    </material>
-    <material name="black">
-	    <color rgba="0 0 0 1"/>
-    </material>
-    <material name="green">
-        <color rgba="0.0 0.8 0.0 1.0"/>
-    </material>
-    <link name="base_link">
-        <!--<visual>
-          <geometry>
-             <box size="0.24 0.24 0.001"/>
-          </geometry>
-          <material name="white"/>
-          <origin rpy="0 0 0" xyz="0 0 0.0005"/>
-          <material>
-            <color rgba="0 0 0.8 1" />
-          </material>
-        </visual> -->
-        <collision>
-          <origin rpy="0 0 0" xyz="0 0 0.0005"/>
-          <geometry>
-            <box size="0.22 0.22 0.001"/>
-          </geometry>
-        </collision>
-    </link>
-    <joint name="base_link_joint" type="fixed">
-        <origin xyz="0 0 0.026" rpy="0 0 -1.5708" />
-        <parent link="base_link" />
-        <child link="base_plate" />
-    </joint>
-    <link name="base_plate">
+<robot name="mobile_robot"
+  xmlns:xacro="http://ros.org/wiki/xacro">
+  <!-- Color Macros -->
+  <material name="blue">
+    <color rgba="0 0 0.8 1"/>
+  </material>
+  <material name="white">
+    <color rgba="1 1 1 1"/>
+  </material>
+  <material name="black">
+    <color rgba="0 0 0 1"/>
+  </material>
+  <material name="green">
+    <color rgba="0.0 0.8 0.0 1.0"/>
+  </material>
+  <!-- Base Properties -->
+  <xacro:property name="body_length" value="0.2" />
+  <xacro:property name="body_width" value="0.1" />
+  <xacro:property name="body_height" value="0.05" />
+  <xacro:property name="ground_offset" value="0.04" />
+  <!-- Wheel Properties -->
+  <xacro:property name="wheelbase" value="0.1" />
+  <xacro:property name="wheel_radius" value="0.04" />
+  <xacro:property name="wheel_length" value="0.02" />
+  <link name="base_link">
     <visual>
-      <origin rpy="1.57079632679 0.0 -91.10079632679" xyz="0.0 0.0 0.015"/>
+      <origin rpy="1.57079632679 0.0 1.57079632679" xyz="0.0 0.0 0.043"/>
       <geometry>
         <mesh filename="package://jetbot_ccai/stl/JetBot-Chassis.stl" scale="0.001 0.001 0.001"/>
@@ -45,17 +33,17 @@
     </visual>
     <collision>
-      <origin rpy="0.0 0.0 0.0" xyz="0.0 0.0 0.015"  />
+      <origin rpy="0.0 0.0 0.0" xyz="0.0 0.0 0.015" />
       <geometry>
         <mesh filename="package://jetbot_ccai/stl/JetBot-Chassis.stl" scale="0.001 0.001 0.001" />
       </geometry>
     </collision>
-    </link>
-    <joint name="right_wheel_joint" type="continuous">
-        <origin xyz="-0.08 -0.06 0.015" rpy="0 0 0" />
-        <parent link="base_plate" />
-        <child link="right_wheel" />
-        <axis xyz="-1 0 0" />
-    </joint>
-    <link name="right_wheel">
+  </link>
+  <joint name="right_wheel_joint" type="continuous">
+    <origin xyz="-0.08 -0.06 0.015" rpy="0 0 0" />
+    <parent link="base_plate" />
+    <child link="right_wheel" />
+    <axis xyz="-1 0 0" />
+  </joint>
+  <link name="right_wheel">
     <visual>
       <origin rpy="0 0 0" xyz="0.127 0.09174 -0.0127"/>
@@ -71,12 +59,12 @@
       </geometry>
     </collision>
-    </link>
-    <joint name="left_wheel_joint" type="continuous">
-        <origin xyz="0.08 -0.06 0.015" rpy="0 0 0" />
-        <parent link="base_plate" />
-        <child link="left_wheel" />
-        <axis xyz="-1 0 0" />
-    </joint>
-    <link name="left_wheel">
+  </link>
+  <joint name="left_wheel_joint" type="continuous">
+    <origin xyz="0.08 -0.06 0.015" rpy="0 0 0" />
+    <parent link="base_plate" />
+    <child link="left_wheel" />
+    <axis xyz="-1 0 0" />
+  </joint>
+  <link name="left_wheel">
     <visual>
       <origin rpy="0 0 0" xyz="-0.1355 0.09174 -0.0127"/>
@@ -92,11 +80,11 @@
       </geometry>
     </collision>
-    </link>
-    <joint name="laser_joint" type="fixed">
-        <origin xyz="0 0.040 0.090" rpy="0 0 1.5708" />
-        <parent link="base_plate" />
-        <child link="laser" />
-    </joint>
-    <link name="laser">
+  </link>
+  <joint name="laser_joint" type="fixed">
+    <origin xyz="0 0.040 0.090" rpy="0 0 1.5708" />
+    <parent link="base_plate" />
+    <child link="laser" />
+  </joint>
+  <link name="laser">
     <visual>
       <origin rpy="0 0 -1.5708" xyz="0.03 -0.248 -0.09"/>
@@ -107,9 +95,9 @@
     </visual>
     <collision>
-      <origin rpy="0 0 0" xyz="0.242 0.084 -0.098"  />
+      <origin rpy="0 0 0" xyz="0.242 0.084 -0.098" />
       <geometry>
         <mesh filename="package://jetbot_ccai/stl/RpLidar.stl" scale="0.001 0.001 0.001" />
       </geometry>
     </collision>
-    </link>
+  </link>
 </robot>
