Commit message: Change frame_id from Rplidar

File: urdf/includes/parts/chassis.xacro (robot description, xacro)
@@ -11,5 +11,5 @@
   <!-- CHASSIS (body) -->
   <xacro:macro name="chassis">
-    <!--link name="base_footprint" /-->
+    <link name="base_footprint" />
     <link name="base_link">
       <visual>
@@ -27,9 +27,10 @@
       </collision>
     </link>
-    <!-- Joint to connect base_link with base_footprint >
+    <!-- Joint to connect base_link with base_footprint -->
     <joint name="base_footprint_joint" type="fixed">
       <parent link="base_footprint"/>
       <child link="base_link" />
-    </joint-->
+      <origin xyz ="0 0 0"/>
+    </joint>
   </xacro:macro>
   <!-- CHASSIS (body) -->

File: urdf/includes/parts/wheels/wheel.xacro (robot description, xacro)
@@ -59,26 +59,26 @@
       <child link="${prefix}_wheelc"/>
     </joint>
-    <!--link name="${prefix}_wheel">
-    <visual>
-    <origin rpy="${pi/2} 0 0" xyz="0 0 0" />
-      <geometry>
-        <cylinder length="${wheelc_len}" radius="${wheelc_r + 0.0065}"/>
-      </geometry>
-      <material name="black"/>
-    </visual>
-    <collision>
-    <origin rpy="${pi/2} 0 0" xyz="0 0 0" />
-      <geometry>
-        <cylinder length="${wheelc_len}" radius="${wheelc_r + 0.0065}"/>
-      </geometry>
-    </collision>
-  </link>
-  <joint name="${prefix}_wheel_joint" type="continuous">
-    <axis xyz="0 1 0"/>
-    <parent link="${prefix}_wheelc"/>
-    <child link="${prefix}_wheel"/>
-    <origin xyz ="0 ${-0.0001*reflect} 0"/>
-  </joint>
-    <xacro:tx prefix="${prefix}" suffix="wheel" /-->
+    <link name="${prefix}_wheel">
+      <visual>
+        <origin rpy="${pi/2} 0 0" xyz="0 0 0" />
+        <geometry>
+          <cylinder length="${wheelc_len}" radius="${wheelc_r + 0.0065}"/>
+        </geometry>
+        <material name="black"/>
+      </visual>
+      <collision>
+        <origin rpy="${pi/2} 0 0" xyz="0 0 0" />
+        <geometry>
+          <cylinder length="${wheelc_len}" radius="${wheelc_r + 0.0065}"/>
+        </geometry>
+      </collision>
+    </link>
+    <joint name="${prefix}_wheel_joint" type="continuous">
+      <axis xyz="0 1 0"/>
+      <parent link="${prefix}_wheelc"/>
+      <child link="${prefix}_wheel"/>
+      <origin xyz ="0 ${-0.0001*reflect} 0"/>
+    </joint>
+    <xacro:tx prefix="${prefix}" suffix="wheel" />
   </xacro:macro>
   <!-- Wheel Macro-->

File: urdf/jetbot.urdf.xacro (robot description, xacro)
@@ -1,4 +1,4 @@
 <?xml version="1.0"?>
-<robot xmlns:xacro="http://www.ros.org/wiki/xacro" name="mobile_robot" >
+<robot xmlns:xacro="http://www.ros.org/wiki/xacro" name="mobile_robot">
   <!-- Xacro arguments for depth camera use -->
   <xacro:arg name="realsense_enable" default="false" />
@@ -37,12 +37,12 @@
   <!-- REALSENSE CAMERA -->
   <xacro:if value="$(arg realsense_enable)">
-    <xacro:sensor_d435 name="realsense_d435" topics_ns="realsense_d435" parent="base_link" publish_pointcloud="$(arg pointcloud_enable)" >
+    <xacro:sensor_d435 name="realsense_d435" topics_ns="realsense_d435" parent="base_link" publish_pointcloud="$(arg pointcloud_enable)">
       <origin xyz="0.077 0 0" rpy="0 0 0" />
     </xacro:sensor_d435>
   </xacro:if>
   <!-- RPLIDAR LASER -->
-  <xacro:if value="$(arg lidar_enable)" >
-    <xacro:sensor_rplidar name="rplidar" topic_ns="scan" parent="pcb_boards" visualize_laser="$(arg visualize_laser)" >
-    <!--xacro:sensor_rplidar name="rplidar" topic_ns="rplidar" parent="pcb_boards" visualize_laser="$(arg visualize_laser)" -->
+  <xacro:if value="$(arg lidar_enable)">
+    <xacro:sensor_rplidar name="rplidar" topic_ns="scan" parent="pcb_boards" visualize_laser="$(arg visualize_laser)">
+      <!--xacro:sensor_rplidar name="rplidar" topic_ns="rplidar" parent="pcb_boards" visualize_laser="$(arg visualize_laser)" -->
       <origin xyz="0 0 0.058" rpy="0 0 0" />
     </xacro:sensor_rplidar >
