Commit message: updates

File: urdf/includes/gazebo/jetbot.gazebo.xacro (robot description, xacro)
@@ -1,4 +1,10 @@
 <?xml version="1.0"?>
 <robot>
+  <!-- Gazebo plugin for ROS Control -->
+  <gazebo>
+    <plugin name="gazebo_ros_control" filename="libgazebo_ros_control.so">
+      <robotNamespace>/</robotNamespace>
+    </plugin>
+  </gazebo>
   <!--Gazebo Camera Plugin-->
   <gazebo reference="camera_lens">

File: urdf/includes/parts/chassis.xacro (robot description, xacro)
@@ -10,27 +10,26 @@
   <!-- Chassis constants -->
   <!-- CHASSIS (body) -->
-  <xacro:macro name="chassis">
-    <link name="base_footprint" />
-    <link name="base_link">
-      <visual>
-        <origin xyz="0 0 ${base_z_offset}"/>
-        <geometry>
-          <box size="${base_len} ${base_width} ${base_height}"/>
-        </geometry>
-        <material name="blue"/>
-      </visual>
-      <collision>
-        <origin xyz="0 0 ${base_z_offset}"/>
-        <geometry>
-          <box size="${base_len} ${base_width} ${base_height}"/>
-        </geometry>
-      </collision>
-    </link>
-    <!-- Joint to connect base_link with base_footprint -->
-    <joint name="base_footprint_joint" type="fixed">
-      <parent link="base_footprint"/>
-      <child link="base_link" />
-      <origin xyz ="0 0 0"/>
-    </joint>
+  <xacro:macro name="chassis" >
+  <link name="base_footprint" />
+  <link name="base_link">
+    <visual>
+      <origin xyz="0 0 ${base_z_offset}"/>
+      <geometry>
+        <box size="${base_len} ${base_width} ${base_height}"/>
+      </geometry>
+      <material name="blue"/>
+    </visual>
+    <collision>
+      <origin xyz="0 0 ${base_z_offset}"/>
+      <geometry>
+        <box size="${base_len} ${base_width} ${base_height}"/>
+      </geometry>
+    </collision>
+  </link>
+  <!-- Joint to connect base_link with base_footprint -->
+  <joint name="base_footprint_joint" type="fixed">
+    <parent link="base_footprint"/>
+    <child link="base_link" />
+  </joint>
   </xacro:macro>
   <!-- CHASSIS (body) -->

File: urdf/includes/parts/wheels/caster.xacro (robot description, xacro)
@@ -12,4 +12,7 @@
   <xacro:property name="caster_ball_mass" value="0.02" />
   <!-- Caster Ball constants -->
+  <!-- Inertia Macro -->
+  <!--xacro:include filename="$(find jetbot_ccai)/urdf/includes/gazebo/inertias.xacro" /-->
+  <!-- Inertia Macro -->
   <!-- Caster Wheel Left and Right Mini Cylinder Macros -->
   <xacro:macro name="caster_minicyl" params="prefix suffix reflect">

File: urdf/includes/parts/wheels/wheel.xacro (robot description, xacro)
@@ -8,77 +8,78 @@
   <xacro:property name="wheelc_len" value="0.015" />
   <xacro:property name="wheelc_r" value = "0.026" />
-  <xacro:property name="wheel_shaft_mass" value = "0.000283495" />
-  <!--0.000283495 0.0028 -->
-  <xacro:property name="wheelc_mass" value = "0.283495" />
-  <!--0.283495 0.00283495 0.0272 -->
-  <xacro:property name="wheel_mass" value = "0.0181" />
-  <!--3.0 0.0181 -->
+  <xacro:property name="wheel_shaft_mass" value = "0.000283495" /> <!--0.000283495 0.0028 -->
+  <xacro:property name="wheelc_mass" value = "0.283495" />  <!--0.283495 0.00283495 0.0272 -->
+  <xacro:property name="wheel_mass" value = "0.0181" />         <!--3.0 0.0181 -->
   <!-- Wheel constants -->
+  <!-- Inertia Macro -->
+  <!--xacro:include filename="$(find jetbot_description)/urdf/includes/gazebo/inertias.xacro" /-->
+  <!-- Inertia Macro -->
   <!-- Wheel Macro-->
   <xacro:macro name="wheel_parts" params="prefix reflect">
-    <link name="${prefix}_wheel_shaft">
-      <visual>
-        <origin xyz="0 0 0" rpy="${pi/2} 0 0"/>
-        <geometry>
-          <cylinder radius="${shaft_r}" length="${shaft_len}" />
-        </geometry>
-        <material name="white"/>
-      </visual>
-      <collision>
-        <origin xyz="0 0 0" rpy="${pi/2} 0 0"/>
-        <geometry>
-          <cylinder radius="${shaft_r}" length="${shaft_len}" />
-        </geometry>
-      </collision>
-    </link>
-    <joint name="base_${prefix}_wheel_shaft_joint" type="fixed">
-      <axis rpy="0 0 0" xyz="0 0 0" />
-      <parent link="base_link"/>
-      <child link="${prefix}_wheel_shaft"/>
-      <origin rpy="0 0 0" xyz="${shaft_xoffset} ${shaft_yoffset*reflect} 0.013" />
-    </joint>
-    <link name="${prefix}_wheelc">
-      <visual>
-        <origin rpy="${pi/2} 0 0"/>
-        <geometry>
-          <cylinder length="${wheelc_len}" radius="${wheelc_r}"/>
-        </geometry>
-        <material name="white"/>
-      </visual>
-      <collision>
-        <origin rpy="${pi/2} 0 0"/>
-        <geometry>
-          <cylinder length="${wheelc_len}" radius="${wheelc_r}"/>
-        </geometry>
-      </collision>
-      <!--xacro:cylinder_inertia mass="${wheelc_mass}" r="${wheelc_r}" h="${wheelc_len}" /-->
-    </link>
-    <joint name="${prefix}_shaft_wheelc_joint" type="fixed">
-      <origin xyz="0 ${reflect*(wheelc_r-0.002)/2} 0"/>
-      <parent link="${prefix}_wheel_shaft"/>
-      <child link="${prefix}_wheelc"/>
-    </joint>
-    <link name="${prefix}_wheel">
-      <visual>
-        <origin rpy="${pi/2} 0 0" xyz="0 0 0" />
-        <geometry>
-          <cylinder length="${wheelc_len}" radius="${wheelc_r + 0.0065}"/>
-        </geometry>
-        <material name="black"/>
-      </visual>
-      <collision>
-        <origin rpy="${pi/2} 0 0" xyz="0 0 0" />
-        <geometry>
-          <cylinder length="${wheelc_len}" radius="${wheelc_r + 0.0065}"/>
-        </geometry>
-      </collision>
-    </link>
-    <joint name="${prefix}_wheel_joint" type="continuous">
-      <axis xyz="0 1 0"/>
-      <parent link="${prefix}_wheelc"/>
-      <child link="${prefix}_wheel"/>
-      <origin xyz ="0 ${-0.0001*reflect} 0"/>
-    </joint>
-    <xacro:tx prefix="${prefix}" suffix="wheel" />
+  <link name="${prefix}_wheel_shaft">
+    <visual>
+      <origin xyz="0 0 0" rpy="${pi/2} 0 0"/>
+      <geometry>
+        <cylinder radius="${shaft_r}" length="${shaft_len}" />
+      </geometry>
+      <material name="white"/>
+    </visual>
+    <collision>
+      <origin xyz="0 0 0" rpy="${pi/2} 0 0"/>
+      <geometry>
+        <cylinder radius="${shaft_r}" length="${shaft_len}" />
+      </geometry>
+    </collision>
+  </link>
+  <joint name="base_${prefix}_wheel_shaft_joint" type="fixed">
+    <axis rpy="0 0 0" xyz="0 0 0" />
+    <parent link="base_link"/>
+    <child link="${prefix}_wheel_shaft"/>
+    <origin rpy="0 0 0" xyz="${shaft_xoffset} ${shaft_yoffset*reflect} 0.013" />
+  </joint>
+  <link name="${prefix}_wheelc">
+    <visual>
+      <origin rpy="${pi/2} 0 0"/>
+      <geometry>
+        <cylinder length="${wheelc_len}" radius="${wheelc_r}"/>
+      </geometry>
+      <material name="white"/>
+    </visual>
+    <collision>
+      <origin rpy="${pi/2} 0 0"/>
+      <geometry>
+        <cylinder length="${wheelc_len}" radius="${wheelc_r}"/>
+      </geometry>
+    </collision>
+    <!--xacro:cylinder_inertia mass="${wheelc_mass}" r="${wheelc_r}" h="${wheelc_len}" /-->
+  </link>
+  <joint name="${prefix}_shaft_wheelc_joint" type="fixed">
+    <origin xyz="0 ${reflect*(wheelc_r-0.002)/2} 0"/>
+    <parent link="${prefix}_wheel_shaft"/>
+    <child link="${prefix}_wheelc"/>
+  </joint>
+  <link name="${prefix}_wheel">
+    <visual>
+    <origin rpy="${pi/2} 0 0" xyz="0 0 0" />
+      <geometry>
+        <cylinder length="${wheelc_len}" radius="${wheelc_r + 0.0065}"/>
+      </geometry>
+      <material name="black"/>
+    </visual>
+    <collision>
+    <origin rpy="${pi/2} 0 0" xyz="0 0 0" />
+      <geometry>
+        <cylinder length="${wheelc_len}" radius="${wheelc_r + 0.0065}"/>
+      </geometry>
+    </collision>
+    <!--xacro:open_cylinder_inertia mass="${wheel_mass}" r1="${wheelc_r}" r2="${wheelc_r + 0.0065}" h="${wheelc_len}" /-->
+  </link>
+  <joint name="${prefix}_wheel_joint" type="continuous">
+    <axis xyz="0 1 0"/>
+    <parent link="${prefix}_wheelc"/>
+    <child link="${prefix}_wheel"/>
+    <origin xyz ="0 ${-0.0001*reflect} 0"/>
+  </joint>
+  <xacro:tx prefix="${prefix}" suffix="wheel" />
   </xacro:macro>
   <!-- Wheel Macro-->
