Commit message: Add URDF models

File: urdf/mobile_robot.urdf.xacro (robot description, xacro)
@@ -1,133 +1,89 @@
 <?xml version="1.0"?>
-<robot name="mobile_robot" xmlns:xacro="http://ros.org/wiki/xacro">
-    <material name="blue">
-	    <color rgba="0 0 0.8 1"/>
-    </material>
-    <material name="white">
-	    <color rgba="1 1 1 1"/>
-    </material>
-    <material name="black">
-	    <color rgba="0 0 0 1"/>
-    </material>
-    <material name="green">
-        <color rgba="0.0 0.8 0.0 1.0"/>
-    </material>
-    <link name="base_link">
-        <!--<visual>
-          <geometry>
-             <box size="0.24 0.24 0.001"/>
-          </geometry>
-          <material name="white"/>
-          <origin rpy="0 0 0" xyz="0 0 0.0005"/>
-          <material>
-            <color rgba="0 0 0.8 1" />
-          </material>
-        </visual> -->
-        <pose>0.0 0.0 0.043 1.57079632679 0.0 1.57079632679</pose>
-			<collision name='collision'>
-				<geometry>
-					<mesh>
-						<scale>0.001 0.001 0.001</scale>
-						<uri>model://jetbot_ccai/gazebo/meshes/JetBot-v3-Chassis.dae</uri>
-					</mesh>
-				</geometry>
-				<surface>
-					<friction>
-						<ode>
-							<mu>0</mu>
-							<mu2>0</mu2>
-							<slip1>1.0</slip1>
-							<slip2>1.0</slip2>
-						</ode>
-					</friction>
-				</surface>
-			</collision>
-    </link>
-    <joint name="F" type="fixed">
-        <origin xyz="0 0 0.026" rpy="0 0 -1.5708" />
-        <parent link="base_link" />
-        <child link="base_plate" />
-    </joint>
-    <link name="base_plate">
-    <visual name='visual'>
-				<geometry>
-					<mesh>
-						<scale>0.001 0.001 0.001</scale>
-						<uri>model://jetbot_ccai/gazebo/meshes/JetBot-v3-Chassis.dae</uri>
-					</mesh>
-				</geometry>
-			</visual>
-    </link>
-    <joint name="right_wheel_joint" type="continuous">
-        <origin xyz="-0.08 -0.06 0.015" rpy="0 0 0" />
-        <parent link="base_plate" />
-        <child link="right_wheel" />
-        <axis xyz="-1 0 0" />
-    </joint>
-    <link name="right_wheel">
-    <pose>0.03 -0.0595 0.03 0.0 0.0 1.57079632679</pose>
-			<collision name="collision">
-				<geometry>
-					<mesh>
-						<scale>0.001 0.001 0.001</scale>
-						<uri>model://jetbot_ccai/gazebo/meshes/JetBot-v3-Wheel.stl</uri>
-					</mesh>
-				</geometry>
-			</collision>
-			<visual name="visual">
-				<geometry>
-					<mesh>
-						<scale>0.001 0.001 0.001</scale>
-						<uri>model://jetbot_ccai/gazebo/meshes/JetBot-v3-Wheel.stl</uri>
-					</mesh>
-				</geometry>
-				<material>
-					<ambient>0.1 0.1 0.1 1</ambient>
-					<diffuse>0.1 0.1 0.1 1</diffuse>
-					<specular>0 0 0 0</specular>
-					<emissive>0 0 0 1</emissive>
-				</material>
-			</visual>
-    </link>
-    <joint name="left_wheel_joint" type="continuous">
-        <origin xyz="0.08 -0.06 0.015" rpy="0 0 0" />
-        <parent link="base_plate" />
-        <child link="left_wheel" />
-        <axis xyz="-1 0 0" />
-    </joint>
-    <link name="left_wheel">
-    <visual>
-      <origin rpy="0 0 0" xyz="0.133 0.059 -0.04"/>
-      <geometry>
-        <mesh filename="package://jetbot_ccai/stl/Wheel.stl" scale="0.001 0.001 0.001"/>
-      </geometry>
-      <material name="black"/>
-    </visual>
-    <collision>
-      <origin rpy="0 0 0" xyz="0.133 0.059 -0.04"/>
-      <geometry>
-        <mesh filename="package://jetbot_ccai/stl/Wheel.stl" scale="0.001 0.001 0.001" />
-      </geometry>
-    </collision>
-    </link>
-    <joint name="laser_joint" type="fixed">
-        <origin xyz="0 0.040 0.090" rpy="0 0 1.5708" />
-        <parent link="base_plate" />
-        <child link="laser" />
-    </joint>
-    <link name="laser">
-    <visual>
-      <origin rpy="0 0 -1.5708" xyz="0.084 -0.242 -0.098"/>
-      <geometry>
-        <mesh filename="package://jetbot_ccai/stl/RpLidar.stl" scale="0.001 0.001 0.001"/>
-      </geometry>
-      <material name="blue"/>
-    </visual>
-    <collision>
-      <origin rpy="0 0 0" xyz="0.242 0.084 -0.098"  />
-      <geometry>
-        <mesh filename="package://mobile_robot_autonomous_navigation/stl/RpLidar.stl" scale="0.001 0.001 0.001" />
-      </geometry>
-    </collision>
-    </link>
+<robot xmlns:xacro="http://www.ros.org/wiki/xacro" name="mobile_robot" >
+  <!-- Xacro arguments for depth camera use -->
+  <xacro:arg name="realsense_enable" default="true" />
+  <xacro:arg name="pointcloud_enable" default="true" />
+  <!-- Xacro arguments for depth lidar use -->
+  <xacro:arg name="lidar_enable" default="true" />
+  <xacro:arg name="visualize_laser" default="true" />
+  <!-- Xacro arguments for imu -->
+  <xacro:arg name="imu_enable" default="true" />
+  <!-- Xacro arguments for gps -->
+  <xacro:arg name="gps_enable" default="true" />
+  <!-- Xacro arguments for ultrasonic -->
+  <xacro:arg name="ultrasonic_enable" default="true" />
+  <!-- All Neccesary Header Files, Macros and Constants -->
+  <xacro:include filename="$(find jetbot_ccai)/urdf/includes.xacro" />
+  <!-- All Neccesary Header FIles, Macros and Constants -->
+  <!-- CHASSIS -->
+  <xacro:chassis />
+  <!-- LEFT WHEEL -->
+  <xacro:wheel_parts prefix="lt" reflect="1" />
+  <!-- RIGHT WHEEL -->
+  <xacro:wheel_parts prefix="rt" reflect="-1" />
+  <!-- FRONT CASTER WHEEL -->
+  <xacro:caster_wheel_parts prefix="front" reflect="1" />
+  <!-- BACK CASTER WHEEL -->
+  <xacro:caster_wheel_parts prefix="back" reflect="-1" />
+  <!-- LEFT ANTENNA -->
+  <xacro:antenna prefix="lt" reflect="1" />
+  <!-- RIGHT ANTENNA -->
+  <xacro:antenna prefix="rt" reflect="-1" />
+  <!-- SENSORS -->
+  <!-- MONOCULAR CAMERA -->
+  <xacro:camera />
+  <!-- BOARDS -->
+  <xacro:pcb />
+  <!-- REALSENSE CAMERA -->
+  <xacro:if value="$(arg realsense_enable)">
+    <xacro:sensor_d435 name="realsense_d435" topics_ns="realsense_d435" parent="base_link" publish_pointcloud="$(arg pointcloud_enable)" >
+      <origin xyz="0.077 0 0" rpy="0 0 0" />
+    </xacro:sensor_d435>
+  </xacro:if>
+  <!-- RPLIDAR LASER -->
+  <xacro:if value="$(arg lidar_enable)" >
+    <xacro:sensor_rplidar name="rplidar" topic_ns="scan" parent="pcb_boards" visualize_laser="$(arg visualize_laser)" >
+    <!--xacro:sensor_rplidar name="rplidar" topic_ns="rplidar" parent="pcb_boards" visualize_laser="$(arg visualize_laser)" -->
+      <origin xyz="0 0 0.058" rpy="0 0 0" />
+    </xacro:sensor_rplidar >
+  </xacro:if>
+  <!-- IMU -->
+  <xacro:if value="$(arg imu_enable)" >
+    <xacro:sensor_imu name="imu" topic_ns="imu" parent="pcb_boards" >
+      <origin xyz="0 0 0.0275" rpy="0 0 0" />
+    </xacro:sensor_imu>
+  </xacro:if>
+  <!-- GPS -->
+  <xacro:if value="$(arg gps_enable)" >
+    <xacro:sensor_gps name="mtk3339" topic_ns="mtk_gps" parent="imu_link" >
+      <origin xyz="-0.044 0 0" rpy="0 0 0" />
+    </xacro:sensor_gps>
+  </xacro:if>
+  <!-- Ultrasonic Sensors -->
+  <xacro:if value="$(arg ultrasonic_enable)" >
+    <xacro:sensor_sonar name="sonar_1" topic_ns="sonar_back_rt" prefix="back_rt" parent="base_link" >
+      <origin xyz="-${base_len/3.5} -${base_width/2} ${base_height/2}" rpy="0 0 -${pi/2}" />
+    </xacro:sensor_sonar>
+    <xacro:sensor_sonar name="sonar_2" topic_ns="sonar_front_rt45" prefix="front_rt45" parent="base_link" >
+      <origin xyz="${base_len/2} -${base_width/2} ${base_height+(base_z_offset)/2}" rpy="0 0 -${pi/4}" />
+    </xacro:sensor_sonar>
+    <xacro:sensor_sonar name="sonar_3" topic_ns="sonar_front" prefix="front" parent="camera_mount_over" >
+      <origin xyz="0 0 0" rpy="0 0 0" />
+    </xacro:sensor_sonar>
+    <xacro:sensor_sonar name="sonar_4" topic_ns="sonar_front_lt45" prefix="front_lt45" parent="base_link" >
+      <origin xyz="${base_len/2} ${base_width/2} ${base_height+(base_z_offset)/2}" rpy="0 0 ${pi/4}" />
+    </xacro:sensor_sonar>
+    <xacro:sensor_sonar name="sonar_5" topic_ns="sonar_back_lt" prefix="back_lt" parent="base_link" >
+      <origin xyz="-${base_len/3.5} ${base_width/2} ${base_height/2}" rpy="0 0 ${pi/2}" />
+    </xacro:sensor_sonar>
+    <xacro:sensor_sonar name="sonar_6" topic_ns="sonar_back_lt45" prefix="back_lt45" parent="base_link" >
+      <origin xyz="-${base_len/2} ${base_width/2} ${base_height+(base_z_offset)/2}" rpy="0 0 ${pi/2 + pi/4}" />
+    </xacro:sensor_sonar>
+    <xacro:sensor_sonar name="sonar_7" topic_ns="sonar_back" prefix="back" parent="base_link" >
+      <origin xyz="-${base_len/2} 0 ${base_height/2}" rpy="0 0 ${pi}" />
+    </xacro:sensor_sonar>
+    <xacro:sensor_sonar name="sonar_8" topic_ns="sonar_back_rt45" prefix="back_rt45" parent="base_link" >
+      <origin xyz="-${base_len/2} -${base_width/2} ${base_height+(base_z_offset)/2}" rpy="0 0 -${pi/2 + pi/4}" />
+    </xacro:sensor_sonar>
+  </xacro:if>
 </robot>

Commit message: Update Model

File: urdf/mobile_robot.urdf.xacro (robot description, xacro)
@@ -1,89 +1,115 @@
 <?xml version="1.0"?>
-<robot xmlns:xacro="http://www.ros.org/wiki/xacro" name="mobile_robot" >
-  <!-- Xacro arguments for depth camera use -->
-  <xacro:arg name="realsense_enable" default="true" />
-  <xacro:arg name="pointcloud_enable" default="true" />
-  <!-- Xacro arguments for depth lidar use -->
-  <xacro:arg name="lidar_enable" default="true" />
-  <xacro:arg name="visualize_laser" default="true" />
-  <!-- Xacro arguments for imu -->
-  <xacro:arg name="imu_enable" default="true" />
-  <!-- Xacro arguments for gps -->
-  <xacro:arg name="gps_enable" default="true" />
-  <!-- Xacro arguments for ultrasonic -->
-  <xacro:arg name="ultrasonic_enable" default="true" />
-  <!-- All Neccesary Header Files, Macros and Constants -->
-  <xacro:include filename="$(find jetbot_ccai)/urdf/includes.xacro" />
-  <!-- All Neccesary Header FIles, Macros and Constants -->
-  <!-- CHASSIS -->
-  <xacro:chassis />
-  <!-- LEFT WHEEL -->
-  <xacro:wheel_parts prefix="lt" reflect="1" />
-  <!-- RIGHT WHEEL -->
-  <xacro:wheel_parts prefix="rt" reflect="-1" />
-  <!-- FRONT CASTER WHEEL -->
-  <xacro:caster_wheel_parts prefix="front" reflect="1" />
-  <!-- BACK CASTER WHEEL -->
-  <xacro:caster_wheel_parts prefix="back" reflect="-1" />
-  <!-- LEFT ANTENNA -->
-  <xacro:antenna prefix="lt" reflect="1" />
-  <!-- RIGHT ANTENNA -->
-  <xacro:antenna prefix="rt" reflect="-1" />
-  <!-- SENSORS -->
-  <!-- MONOCULAR CAMERA -->
-  <xacro:camera />
-  <!-- BOARDS -->
-  <xacro:pcb />
-  <!-- REALSENSE CAMERA -->
-  <xacro:if value="$(arg realsense_enable)">
-    <xacro:sensor_d435 name="realsense_d435" topics_ns="realsense_d435" parent="base_link" publish_pointcloud="$(arg pointcloud_enable)" >
-      <origin xyz="0.077 0 0" rpy="0 0 0" />
-    </xacro:sensor_d435>
-  </xacro:if>
-  <!-- RPLIDAR LASER -->
-  <xacro:if value="$(arg lidar_enable)" >
-    <xacro:sensor_rplidar name="rplidar" topic_ns="scan" parent="pcb_boards" visualize_laser="$(arg visualize_laser)" >
-    <!--xacro:sensor_rplidar name="rplidar" topic_ns="rplidar" parent="pcb_boards" visualize_laser="$(arg visualize_laser)" -->
-      <origin xyz="0 0 0.058" rpy="0 0 0" />
-    </xacro:sensor_rplidar >
-  </xacro:if>
-  <!-- IMU -->
-  <xacro:if value="$(arg imu_enable)" >
-    <xacro:sensor_imu name="imu" topic_ns="imu" parent="pcb_boards" >
-      <origin xyz="0 0 0.0275" rpy="0 0 0" />
-    </xacro:sensor_imu>
-  </xacro:if>
-  <!-- GPS -->
-  <xacro:if value="$(arg gps_enable)" >
-    <xacro:sensor_gps name="mtk3339" topic_ns="mtk_gps" parent="imu_link" >
-      <origin xyz="-0.044 0 0" rpy="0 0 0" />
-    </xacro:sensor_gps>
-  </xacro:if>
-  <!-- Ultrasonic Sensors -->
-  <xacro:if value="$(arg ultrasonic_enable)" >
-    <xacro:sensor_sonar name="sonar_1" topic_ns="sonar_back_rt" prefix="back_rt" parent="base_link" >
-      <origin xyz="-${base_len/3.5} -${base_width/2} ${base_height/2}" rpy="0 0 -${pi/2}" />
-    </xacro:sensor_sonar>
-    <xacro:sensor_sonar name="sonar_2" topic_ns="sonar_front_rt45" prefix="front_rt45" parent="base_link" >
-      <origin xyz="${base_len/2} -${base_width/2} ${base_height+(base_z_offset)/2}" rpy="0 0 -${pi/4}" />
-    </xacro:sensor_sonar>
-    <xacro:sensor_sonar name="sonar_3" topic_ns="sonar_front" prefix="front" parent="camera_mount_over" >
-      <origin xyz="0 0 0" rpy="0 0 0" />
-    </xacro:sensor_sonar>
-    <xacro:sensor_sonar name="sonar_4" topic_ns="sonar_front_lt45" prefix="front_lt45" parent="base_link" >
-      <origin xyz="${base_len/2} ${base_width/2} ${base_height+(base_z_offset)/2}" rpy="0 0 ${pi/4}" />
-    </xacro:sensor_sonar>
-    <xacro:sensor_sonar name="sonar_5" topic_ns="sonar_back_lt" prefix="back_lt" parent="base_link" >
-      <origin xyz="-${base_len/3.5} ${base_width/2} ${base_height/2}" rpy="0 0 ${pi/2}" />
-    </xacro:sensor_sonar>
-    <xacro:sensor_sonar name="sonar_6" topic_ns="sonar_back_lt45" prefix="back_lt45" parent="base_link" >
-      <origin xyz="-${base_len/2} ${base_width/2} ${base_height+(base_z_offset)/2}" rpy="0 0 ${pi/2 + pi/4}" />
-    </xacro:sensor_sonar>
-    <xacro:sensor_sonar name="sonar_7" topic_ns="sonar_back" prefix="back" parent="base_link" >
-      <origin xyz="-${base_len/2} 0 ${base_height/2}" rpy="0 0 ${pi}" />
-    </xacro:sensor_sonar>
-    <xacro:sensor_sonar name="sonar_8" topic_ns="sonar_back_rt45" prefix="back_rt45" parent="base_link" >
-      <origin xyz="-${base_len/2} -${base_width/2} ${base_height+(base_z_offset)/2}" rpy="0 0 -${pi/2 + pi/4}" />
-    </xacro:sensor_sonar>
-  </xacro:if>
+<robot name="mobile_robot" xmlns:xacro="http://ros.org/wiki/xacro">
+    <material name="blue">
+	    <color rgba="0 0 0.8 1"/>
+    </material>
+    <material name="white">
+	    <color rgba="1 1 1 1"/>
+    </material>
+    <material name="black">
+	    <color rgba="0 0 0 1"/>
+    </material>
+    <material name="green">
+        <color rgba="0.0 0.8 0.0 1.0"/>
+    </material>
+    <link name="base_link">
+        <!--<visual>
+          <geometry>
+             <box size="0.24 0.24 0.001"/>
+          </geometry>
+          <material name="white"/>
+          <origin rpy="0 0 0" xyz="0 0 0.0005"/>
+          <material>
+            <color rgba="0 0 0.8 1" />
+          </material>
+        </visual> -->
+        <collision>
+          <origin rpy="0 0 0" xyz="0 0 0.0005"/>
+          <geometry>
+            <box size="0.22 0.22 0.001"/>
+          </geometry>
+        </collision>
+    </link>
+    <joint name="base_link_joint" type="fixed">
+        <origin xyz="0 0 0.026" rpy="0 0 -1.5708" />
+        <parent link="base_link" />
+        <child link="base_plate" />
+    </joint>
+    <link name="base_plate">
+    <visual>
+      <origin rpy="1.57079632679 0.0 1.57079632679" xyz="0.0 0.0 0.043"/>
+      <geometry>
+        <mesh filename="package://jetbot_ccai/stl/JetBot-Chassis.stl" scale="0.001 0.001 0.001"/>
+      </geometry>
+      <material name="white"/>
+    </visual>
+    <collision>
+      <origin rpy="0 0 0" xyz="0.03 0 -0.026"  />
+      <geometry>
+        <mesh filename="package://jetbot_ccai/stl/JetBot-Chassis.stl" scale="0.001 0.001 0.001" />
+      </geometry>
+    </collision>
+    </link>
+    <joint name="right_wheel_joint" type="continuous">
+        <origin xyz="-0.08 -0.06 0.015" rpy="0 0 0" />
+        <parent link="base_plate" />
+        <child link="right_wheel" />
+        <axis xyz="-1 0 0" />
+    </joint>
+    <link name="right_wheel">
+    <visual>
+      <origin rpy="0 0 0" xyz="0.11 0.059 -0.04"/>
+      <geometry>
+        <mesh filename="package://jetbot_ccai/stl/Wheel.stl" scale="0.001 0.001 0.001"/>
+      </geometry>
+      <material name="black"/>
+    </visual>
+    <collision>
+      <origin rpy="0 0 0" xyz="0.11 0.059 -0.04"/>
+      <geometry>
+        <mesh filename="package://jetbot_ccai/stl/Wheel.stl" scale="0.001 0.001 0.001" />
+      </geometry>
+    </collision>
+    </link>
+    <joint name="left_wheel_joint" type="continuous">
+        <origin xyz="0.08 -0.06 0.015" rpy="0 0 0" />
+        <parent link="base_plate" />
+        <child link="left_wheel" />
+        <axis xyz="-1 0 0" />
+    </joint>
+    <link name="left_wheel">
+    <visual>
+      <origin rpy="0 0 0" xyz="0.133 0.059 -0.04"/>
+      <geometry>
+        <mesh filename="package://jetbot_ccai/stl/Wheel.stl" scale="0.001 0.001 0.001"/>
+      </geometry>
+      <material name="black"/>
+    </visual>
+    <collision>
+      <origin rpy="0 0 0" xyz="0.133 0.059 -0.04"/>
+      <geometry>
+        <mesh filename="package://jetbot_ccai/stl/Wheel.stl" scale="0.001 0.001 0.001" />
+      </geometry>
+    </collision>
+    </link>
+    <joint name="laser_joint" type="fixed">
+        <origin xyz="0 0.040 0.090" rpy="0 0 1.5708" />
+        <parent link="base_plate" />
+        <child link="laser" />
+    </joint>
+    <link name="laser">
+    <visual>
+      <origin rpy="0 0 -1.5708" xyz="0.084 -0.242 -0.098"/>
+      <geometry>
+        <mesh filename="package://jetbot_ccai/stl/RpLidar.stl" scale="0.001 0.001 0.001"/>
+      </geometry>
+      <material name="blue"/>
+    </visual>
+    <collision>
+      <origin rpy="0 0 0" xyz="0.242 0.084 -0.098"  />
+      <geometry>
+        <mesh filename="package://jetbot_ccai/stl/RpLidar.stl" scale="0.001 0.001 0.001" />
+      </geometry>
+    </collision>
+    </link>
 </robot>

Commit message: Update Urdf model

File: urdf/mobile_robot.urdf.xacro (robot description, xacro)
@@ -38,12 +38,12 @@
     <link name="base_plate">
     <visual>
-      <origin rpy="1.57079632679 0.0 1.57079632679" xyz="0.0 0.0 0.043"/>
+      <origin rpy="1.57079632679 0.0 -91.10079632679" xyz="0.0 0.0 0.015"/>
       <geometry>
         <mesh filename="package://jetbot_ccai/stl/JetBot-Chassis.stl" scale="0.001 0.001 0.001"/>
       </geometry>
-      <material name="white"/>
+      <material name="green"/>
     </visual>
     <collision>
-      <origin rpy="0 0 0" xyz="0.03 0 -0.026"  />
+      <origin rpy="0.0 0.0 0.0" xyz="0.0 0.0 0.015"  />
       <geometry>
         <mesh filename="package://jetbot_ccai/stl/JetBot-Chassis.stl" scale="0.001 0.001 0.001" />
@@ -59,14 +59,14 @@
     <link name="right_wheel">
     <visual>
-      <origin rpy="0 0 0" xyz="0.11 0.059 -0.04"/>
+      <origin rpy="0 0 0" xyz="0.127 0.09174 -0.0127"/>
       <geometry>
-        <mesh filename="package://jetbot_ccai/stl/Wheel.stl" scale="0.001 0.001 0.001"/>
+        <mesh filename="package://jetbot_ccai/stl/JetBot-Wheel.stl" scale="0.001 0.001 0.001"/>
       </geometry>
       <material name="black"/>
     </visual>
     <collision>
-      <origin rpy="0 0 0" xyz="0.11 0.059 -0.04"/>
+      <origin rpy="0 0 0" xyz="0.127 0.09174 -0.0127"/>
       <geometry>
-        <mesh filename="package://jetbot_ccai/stl/Wheel.stl" scale="0.001 0.001 0.001" />
+        <mesh filename="package://jetbot_ccai/stl/JetBot-Wheel.stl" scale="0.001 0.001 0.001" />
       </geometry>
     </collision>
@@ -80,14 +80,14 @@
     <link name="left_wheel">
     <visual>
-      <origin rpy="0 0 0" xyz="0.133 0.059 -0.04"/>
+      <origin rpy="0 0 0" xyz="-0.1355 0.09174 -0.0127"/>
       <geometry>
-        <mesh filename="package://jetbot_ccai/stl/Wheel.stl" scale="0.001 0.001 0.001"/>
+        <mesh filename="package://jetbot_ccai/stl/JetBot-Wheel.stl" scale="0.001 0.001 0.001"/>
       </geometry>
       <material name="black"/>
     </visual>
     <collision>
-      <origin rpy="0 0 0" xyz="0.133 0.059 -0.04"/>
+      <origin rpy="0 0 0" xyz="-0.1355 0.09174 -0.0127"/>
       <geometry>
-        <mesh filename="package://jetbot_ccai/stl/Wheel.stl" scale="0.001 0.001 0.001" />
+        <mesh filename="package://jetbot_ccai/stl/JetBot-Wheel.stl" scale="0.001 0.001 0.001" />
       </geometry>
     </collision>
@@ -100,5 +100,5 @@
     <link name="laser">
     <visual>
-      <origin rpy="0 0 -1.5708" xyz="0.084 -0.242 -0.098"/>
+      <origin rpy="0 0 -1.5708" xyz="0.03 -0.248 -0.09"/>
       <geometry>
         <mesh filename="package://jetbot_ccai/stl/RpLidar.stl" scale="0.001 0.001 0.001"/>

Commit message: Turning RpLidar

File: urdf/mobile_robot.urdf.xacro (robot description, xacro)
@@ -45,5 +45,5 @@
     <xacro:sensor_rplidar name="rplidar" topic_ns="scan" parent="pcb_boards" visualize_laser="$(arg visualize_laser)" >
     <!--xacro:sensor_rplidar name="rplidar" topic_ns="rplidar" parent="pcb_boards" visualize_laser="$(arg visualize_laser)" -->
-      <origin xyz="0 0 0.058" rpy="0 0 0" />
+      <origin xyz="0 0 0.058" rpy="0 0 3.14" />
     </xacro:sensor_rplidar >
   </xacro:if>
